File: winch-pcb/winch.kicad_pcb (KiCad board)
At the start: 2 copper layers, 70 x 60 mm, 15 parts, among them M1 Motor_DC, Q1 IRLB8721, SW1 SW_SPST, U1 Sparkfun_TB6612, U2 Sparkfun_ESP32, U3 LM1117-3.3

Commit message: created pdfs and pngs of schmatic and board
Other:
- board text added: "+"
- board text added: "short these two if not in use"
Changed lines of the file:
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@@
   (general
     (thickness 1.6)
-    (drawings 23)
+    (drawings 30)
     (tracks 63)
     (zones 0)
@@
   )
   (page A4)
+  (title_block
+    (title "Volaser Winch PCB")
+    (company EAWAG)
+    (comment 1 "Matt Grau")
+  )
   (layers
     (0 F.Cu signal)
@@
     (47 F.CrtYd user)
     (48 B.Fab user)
-    (49 F.Fab user)
+    (49 F.Fab user hide)
   )
   (setup
@@
     (visible_elements FFFFFF7F)
     (pcbplotparams
-      (layerselection 0x010fc_ffffffff)
+      (layerselection 0x013fc_ffffffff)
       (usegerberextensions false)
       (usegerberattributes false)
@@
       (padsonsilk false)
       (subtractmaskfromsilk false)
-      (outputformat 1)
+      (outputformat 4)
       (mirror false)
       (drillshape 0)
       (scaleselection 1)
-      (outputdirectory "gerber/"))
+      (outputdirectory "./"))
   )
   (net 0 "")
@@
       (xy -8.2677 1.1176) (xy -8.2042 1.1176) (xy -8.2042 2.1082)) (layer F.SilkS) (width 0.01))
   )
+  (gr_text "short these\ntwo if not in\nuse" (at 121.5 96) (layer F.SilkS)
+    (effects (font (size 0.75 0.75) (thickness 0.15)) (justify left))
+  )
+  (gr_line (start 123 93) (end 123 89) (layer F.SilkS) (width 1))
+  (gr_line (start 125.5 93) (end 123 93) (layer F.SilkS) (width 1))
+  (gr_line (start 125.5 89) (end 125.5 93) (layer F.SilkS) (width 1))
+  (gr_text + (at 104 113) (layer F.SilkS)
+    (effects (font (size 1.5 1.5) (thickness 0.3)))
+  )
+  (gr_text + (at 125 76) (layer F.SilkS)
+    (effects (font (size 1.5 1.5) (thickness 0.3)))
+  )
+  (gr_text + (at 113 76) (layer F.SilkS)
+    (effects (font (size 1.5 1.5) (thickness 0.3)))
+  )
   (dimension 60 (width 0.3) (layer Dwgs.User)
