File: winch-pcb/winch.sch (KiCad schematic (older format))
At the start: 14 parts, among them M1 Motor_DC, Q1 IRLB8721, SW1 SW_SPST, U1 Sparkfun_TB6612, U2 Sparkfun_ESP32, U3 LM1117-3.3

Commit message: created pdfs and pngs of schmatic and board
Other:
- note added: "4 mm mounting holes"
- moved on the sheet: BT1, C1, C2, C3, H1, H2, H3, H4, M1, Q1, SW1, U1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
